Commit message: changes to slam and sim

File: project_ros_ws/src/simulation/urdf/scout-laser.urdf.xacro (robot description, xacro)
@@ -193,4 +193,42 @@
     </sensor>
   </gazebo>
+  <!-- IMU -->
+  <link name="imu_link">
+    <inertial>
+      <pose>0 0 0 0 0 0</pose>
+      <mass value="0.001"/>
+      <inertia ixx="0.000001" ixy="0" ixz="0" iyy="0.000001" iyz="0" izz="0.000001"/>
+    </inertial>
+    <visual>
+      <geometry>
+        <box size="0.01 0.01 0.01"/>
+      </geometry>
+      <material name="Red">
+        <color rgba="0.5 0 0 1"/>
+      </material>
+    </visual>
+  </link>
+  <joint name="imu_joint" type="fixed">
+    <parent link="base_link"/>
+    <child link="imu_link"/>
+    <origin xyz="0 0 0" rpy="0 0 0"/>
+  </joint>
+  <gazebo reference='imu_link'>
+    <sensor name='robot_imu' type='imu'>
+      <always_on>true</always_on>
+      <update_rate>20</update_rate>
+      <visualize>false</visualize>
+      <plugin filename='libgazebo_ros_imu_sensor.so' name='imu_sensor'>
+        <topicName>imu_data</topicName>
+        <ros>
+          <namespace>/</namespace>
+          <remapping>~/out:=imu_data</remapping>
+        </ros>
+        <frameName>robot_imu</frameName>
+        <output_type>sensor_msgs/Imu</output_type>
+        <initial_orientation_as_reference>false</initial_orientation_as_reference>
+      </plugin>
+    </sensor>
+  </gazebo>
   <!-- Left wheel -->
   <gazebo reference="left_wheel_link">
